File: pro_micro_programmer.kicad_pcb (KiCad board)
At the start: 2 copper layers, 17.8 x 35.6 mm, 5 parts, among them J1 Conn_01x12, J2 Conn_01x12, J3 Conn_02x03

Commit message: [docs]fix typo
Parts:
- added G***: LOGO, lib:promicro_programmer_logo, B.Cu at (146.1, 94.0)
- added G***: LOGO, logo_silk:logo_toms_85x40_silk, B.Cu at (146.7, 106.7)
