File: pro_micro_programmer_panelize.kicad_pcb (KiCad board)
At the start: 2 copper layers, 94 x 85.1 mm, 73 parts, among them J1 Conn_01x12, J2 Conn_01x12, J3 Conn_02x03

Commit message: [add]add silk
Other:
- board text added: "▲USB"
